File: schematic.kicad_sch (KiCad schematic)
At the start: 0 parts

Commit message: feat(ui/cad): suite esquematica CAD industrial 5 folhas, telemetria 18 canais e correcao do pedal
- Implementa Suite Esquematica CAD Industrial interativa com 5 folhas integradas inline
- Corrige telemetria reativa do acelerador (simulacao e modo real com feedback imediato)
- Adiciona 18 canais de telemetria grafica no Chart.js com estatisticas de pico
- Aprimora esquematico vetorial com conexoes de gate rapidas (1N4148), barramento PWM, shunts Kelvin e CAN isolado
- Adiciona suites de testes automatizados e validacao de console no Playwright
Parts:
- added C1, C2: 470uF, symbol MotorCtrl:C
- added F1: 50A, symbol MotorCtrl:R
- added Q1, Q2, Q3, Q4, Q5, Q6: IPP65R600P7, symbol MotorCtrl:Q_NMOS
- added Rsh_U, Rsh_V, Rsh_W: 0.001R, symbol MotorCtrl:R
- added U1: ESP32-WROOM-32E, symbol MotorCtrl:ESP32
- added U2: DRV8302, symbol MotorCtrl:DRV8302
Connections:
- new net: Q1.1 (G), Q2.1 (G)
- new net: Q3.1 (G), Q4.1 (G), U2.12 (GLC), U2.13 (DVDD)
- new net: Q5.1 (G), Q6.1 (G), U2.10 (GLB), U2.11 (GHC)
- new net: U1.7 (GPIO36), U1.8 (GPIO39), U1.9 (GPIO34), U2.5 (nFAULT), U2.6 (GND)
- new net +400V: C1.1, C1.2, C2.1, C2.2, F1.1, F1.2, Q1.2 (D), Q1.3 (S), Q2.2 (D), Q2.3 (S), Q3.2 (D), Q3.3 (S), Q4.2 (D), Q4.3 (S), Q5.2 (D), Q5.3 (S), Q6.2 (D), Q6.3 (S), Rsh_U.1, Rsh_V.1, Rsh_W.1
- new net GND: Rsh_U.2, Rsh_V.2, Rsh_W.2
Other:
- note removed: "Components: C1, Q1-Q3, Q4-Q6, U1, U2"
- note removed: "PMSM/BLDC 3-Phase Motor Controller"
- note removed: "Production-Grade Design | 57 Components | KiCad 9.0"
- company: OpenCode -> (none)
- title: Universal PMSM/BLDC Motor Controller -> (none)
