File: schematic_real.kicad_sch (KiCad schematic)
At the start: 53 parts, among them Q1-Q3 600V 100A, Q4-Q6 600V 100A, U1 240MHz Xtensa, U2 3-phase motor driver

Commit message: feat(ui/cad): suite esquematica CAD industrial 5 folhas, telemetria 18 canais e correcao do pedal
- Implementa Suite Esquematica CAD Industrial interativa com 5 folhas integradas inline
- Corrige telemetria reativa do acelerador (simulacao e modo real com feedback imediato)
- Adiciona 18 canais de telemetria grafica no Chart.js com estatisticas de pico
- Aprimora esquematico vetorial com conexoes de gate rapidas (1N4148), barramento PWM, shunts Kelvin e CAN isolado
- Adiciona suites de testes automatizados e validacao de console no Playwright
Parts:
- removed LDO_regulator: TI LM7805 or similar, symbol Power_Management:LM7805
- added CORRECAO 1: Fase 1 (prototipo) opera em bancada 12-48V. DRV8302 e 8-60V PVDD - nao suporta link de 400V. Para 400V (Fase 2) usar drivers HV (UCC21520/IR2184 x3) + MOSFETs 600V alta corrente (IXFN100N60P/SiC) + cooling ativo.: (no value), symbol Device:R
- added CORRECAO 2: IPP65R600P7 e 600V/~6A/0.6Ohm - NAO e 100A/0.01Ohm como a BOM antiga afirmava. Para bancada 48V/30A usar IRFB4110 (100V/180A/4.5mOhm).: (no value), symbol Device:R
- added CORRECAO 3: LM7805 removido (max 35V input). O buck integrado do DRV8302 (TPS54160, 60V/1.5A) supre 5V/3.3V do MCU. LM2596HV listado como opcional.: (no value), symbol Device:R
- added Fase 2 (400V/50kW+): drivers HV + SiC + liquid cooling + EMC - fora desta BOM.: (no value), symbol Device:R
- added Heatsink recalculado para bancada 30A: ~25W total (conducao 3.2W + comutacao ~1W por MOSFET) - passivo ok.: (no value), symbol Device:R
- C1: value 470µF 450V ESL 20mOhm -> 470uF 450V
- C_boot1, C_boot2, C_boot3: value 10µF 50V -> 10uF 50V
- Cable_motor: value 6mm² shielded -> 6mm2 shielded
- Cable_power: value 6mm² 400V rated -> 6mm2 silicone 400V rated
- Capacitor_5V: value 100µF 16V -> 100uF 16V
- Cfilter_1: value 100µF 10V -> 100uF 10V
- Connector_XT60: value XT60 -> XT60 (par)
- Fasteners: value A2-70 Stainless -> Stainless
- Hall_A, Hall_B, Hall_C: value Linear A3144 -> A3144
- Heatsink_main: value 300x200x10mm 0.3K/W -> 300x200x10mm
- Lfilter_u, Lfilter_v, Lfilter_w: value 1µH 600MHz -> 1uH 600MHz
- Lvcc: value 10µH -> 10uH
- Q1-Q3, Q4-Q6: value 600V 100A -> 100V 180A 4.5mOhm
- R_shunt_u, R_shunt_v, R_shunt_w: value 0.001 Ohm 10W 2% -> 0.001 Ohm 2% 3W
- U2: value 3-phase motor driver -> 3-phase driver 8-60V
